Commit message: update

File: src/go2_description/xacro/leg.xacro (robot description, xacro)
@@ -44,5 +44,5 @@
         </xacro:if>
         <geometry>
-          <mesh filename="file://$(find go2_description)/meshes/hip.dae" scale="1 1 1"/>
+          <mesh filename="package://go2_description/meshes/hip.dae" scale="1 1 1"/>
         </geometry>
       </visual>
@@ -76,8 +76,8 @@
         <geometry>
           <xacro:if value="${mirror_dae == True}">
-            <mesh filename="file://$(find go2_description)/meshes/thigh.dae" scale="1 1 1"/>
+            <mesh filename="package://go2_description/meshes/thigh.dae" scale="1 1 1"/>
           </xacro:if>
           <xacro:if value="${mirror_dae == False}">
-            <mesh filename="file://$(find go2_description)/meshes/thigh_mirror.dae" scale="1 1 1"/>
+            <mesh filename="package://go2_description/meshes/thigh_mirror.dae" scale="1 1 1"/>
           </xacro:if>
         </geometry>
@@ -111,5 +111,5 @@
         <origin rpy="0 0 0" xyz="0 0 0"/>
         <geometry>
-          <mesh filename="file://$(find go2_description)/meshes/calf.dae" scale="1 1 1"/>
+          <mesh filename="package://go2_description/meshes/calf.dae" scale="1 1 1"/>
         </geometry>
       </visual>

File: src/go2_description/xacro/robot.xacro (robot description, xacro)
@@ -52,5 +52,5 @@
       <origin rpy="0 0 0" xyz="0 0 0"/>
       <geometry>
-        <mesh filename="file://$(find go2_description)/meshes/trunk.dae" scale="1 1 1"/>
+        <mesh filename="package://go2_description/meshes/trunk.dae" scale="1 1 1"/>
       </geometry>
       <!-- <material name="orange"/> -->
